File: ADC.kicad_sch (KiCad schematic)
At the start: 0 parts

Commit message: updated cell schematic
Parts:
- added IC1: MCP3304-CI_SL, SOIC127P600X175-16N, symbol MCP3304-CI_SL:MCP3304-CI_SL
Changed lines of the file:
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@@
 	(generator_version "8.0")
 	(paper "A4")
+	(symbol
+		(lib_id "MCP3304-CI_SL:MCP3304-CI_SL")
+		(at 144.145 100.965 0)
+		(unit 1)
+		(exclude_from_sim no)
+		(in_bom yes)
+		(on_board yes)
+		(dnp no)
+		(fields_autoplaced yes)
+		(property "Reference" "IC1"
+			(at 160.655 93.98 0)
+			(effects
+				(font
+					(size 1.27 1.27)
+				)
+			)
+		)
+		(property "Value" "MCP3304-CI_SL"
+			(at 160.655 96.52 0)
+			(effects
+				(font
+					(size 1.27 1.27)
+				)
+			)
+		)
+		(property "Footprint" "SOIC127P600X175-16N"
+			(at 173.355 195.885 0)
+			(effects
+				(font
+					(size 1.27 1.27)
+				)
+				(justify left top)
+				(hide yes)
+			)
+		)
+		(property "Datasheet" "http://ww1.microchip.com/downloads/en/DeviceDoc/21697F.pdf"
+			(at 173.355 295.885 0)
+			(effects
+				(font
+					(size 1.27 1.27)
+				)
+				(justify left top)
+				(hide yes)
+			)
+		)
+		(property "Description" "13-bit ADC,Diff I/P,4chan,MCP3304-CI/SL"
+			(at 144.145 100.965 0)
+			(effects
+				(font
+					(size 1.27 1.27)
+				)
+				(hide yes)
+			)
+		)
+		(property "Height" "1.75"
+			(at 173.355 495.885 0)
+			(effects
+				(font
+					(size 1.27 1.27)
+				)
+				(justify left top)
+				(hide yes)
+			)
+		)
+		(property "Mouser Part Number" "579-MCP3304-CI/SL"
+			(at 173.355 595.885 0)
+			(effects
+				(font
+					(size 1.27 1.27)
+				)
+				(justify left top)
+				(hide yes)
+			)
+		)
+		(property "Mouser Price/Stock" "https://www.mouser.co.uk/ProductDetail/Microchip-Technology/MCP3304-CI-SL?qs=e4wS3D8CKP50gmfqQ11PGg%3D%3D"
+			(at 173.355 695.885 0)
+			(effects
+				(font
+					(size 1.27 1.27)
+				)
+				(justify left top)
+				(hide yes)
+			)
+		)
+		(property "Manufacturer_Name" "Microchip"
+			(at 173.355 795.885 0)
+			(effects
+				(font
+					(size 1.27 1.27)
+				)
+				(justify left top)
+				(hide yes)
+			)
+		)
+		(property "Manufacturer_Part_Number" "MCP3304-CI/SL"
+			(at 173.355 895.885 0)
+			(effects
+				(font
+					(size 1.27 1.27)
+				)
+				(justify left top)
+				(hide yes)
+			)
+		)
+		(pin "5"
+		)
+		(pin "6"
+		)
+		(pin "13"
+		)
+		(pin "8"
+		)
+		(pin "1"
+		)
+		(pin "11"
+		)
+		(pin "16"
+		)
+		(pin "3"
+		)
+		(pin "10"
+		)
+		(pin "14"
+		)
+		(pin "2"
+		)
+		(pin "7"
+		)
+		(pin "12"
+		)
+		(pin "4"
+		)
+		(pin "9"
+		)
+		(pin "15"
+		)
+		(instances
+			(project "Cell-Characterization-Board"
+				(path "/8cf78a1b-eb7a-4166-aa75-ad898a030304/c2cf6403-ef36-48a6-adae-c490417c2e39"
+					(reference "IC1")
+					(unit 1)
+				)
+			)
+		)
+	)
 )
